File: fuenteDC.kicad_pcb (KiCad board)
At the start: 2 copper layers, 96.5 x 80 mm, 15 parts

Commit message: update pcb
Parts:
- removed 5VUSB1: USB3_A, Connector_USB:USB_A_CONNFLY_DS1095-WNR0
- added USB1: Screw_Terminal_01x02, TerminalBlock:TerminalBlock_bornier-2_P5.08mm, F.Cu at (101.6, 61.0)
- Button5V1: value Screw_Terminal_01x02 -> Screw_Terminal_01x03; footprint TerminalBlock:TerminalBlock_bornier-2_P5.08mm -> TerminalBlock:TerminalBlock_bornier-3_P5.08mm
- moved Potentiometer1 38.2 mm to (152.4, 101.6), turned to 180 degrees
- moved Button5V1 14.4 mm to (127.0, 101.6), turned to 180 degrees
- moved Transformer1 12.0 mm to (172.7, 66.0)
- moved Rectifier1 9.67 mm to (147.3, 58.4)
- moved 5VRegulator1 9.03 mm to (129.5, 88.9)
- moved REF3.2mmM3 8.13 mm to (99.1, 109.2)
- moved REF3.2mmM3 7.41 mm to (172.7, 109.2)
- moved 5VVoltamperimeter1 6.84 mm to (101.6, 96.5)
- moved REF3.2mmM3 5.08 mm to (99.1, 45.7)
- moved Fuse1 3.81 mm to (154.9, 45.7)
- moved REF3.2mmM3 3.81 mm to (172.7, 45.7)
Connections:
- Button5V1 pad 2: 5VB -> GND
Routing:
- net 5VVA: track 68.1 -> 112.1 mm
- net GNDUSB: track 27.6 -> 10.2 mm
- net 5V: track 76.6 -> 62.2 mm
- net 5VB: track 57.9 -> 47.0 mm
- net 5VOut: track 53.6 -> 46.3 mm
- net Net-(Fuse1-Pad1): track 21.5 -> 15.9 mm
- net ROut: track 64.7 -> 59.0 mm
- net 12V: track 36.0 -> 30.6 mm
- net 0: track 17.9 -> 16.1 mm
Other:
- board size 96.5 x 80 mm -> 86.4 x 77.5 mm
