File: fuenteDC.kicad_sch (KiCad schematic)
At the start: 11 parts

Commit message: update pcb
Parts:
- removed 5VUSB1: USB3_A, Connector_USB:USB_A_CONNFLY_DS1095-WNR0, symbol Connector:USB3_A
- removed Button5V1: Screw_Terminal_01x02, TerminalBlock:TerminalBlock_bornier-2_P5.08mm, symbol Connector:Screw_Terminal_01x02
- added Button5V1: Screw_Terminal_01x03, TerminalBlock:TerminalBlock_bornier-3_P5.08mm, symbol Connector:Screw_Terminal_01x03
- added USB1: Screw_Terminal_01x02, TerminalBlock:TerminalBlock_bornier-2_P5.08mm, symbol Connector:Screw_Terminal_01x02
Connections:
- net 5V: now also Button5V1.1 (Pin_1)
- net 5VB: now also Button5V1.3 (Pin_3)
- net 5VVA: now also USB1.1 (Pin_1)
- net GND: now also Button5V1.2 (Pin_2)
- net GNDUSB: now also USB1.2 (Pin_2)
Changed lines of the file:
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@@
+    )
+  )
+  (global_label "5VB" (shape input) (at 209.55 96.52 180) (fields_autoplaced)
+    (effects (font (size 1.27 1.27)) (justify right))
+    (property "Intersheet References" "${INTERSHEET_REFS}" (id 0) (at 203.5688 96.4406 0)
+      (effects (font (size 1.27 1.27)) (justify right) hide)
     )
   )
@@
     )
   )
-  (global_label "5VB" (shape input) (at 209.55 95.25 180) (fields_autoplaced)
-    (effects (font (size 1.27 1.27)) (justify right))
-    (property "Intersheet References" "${INTERSHEET_REFS}" (id 0) (at 203.5688 95.1706 0)
+  (global_label "5V" (shape input) (at 209.55 91.44 180) (fields_autoplaced)
+    (effects (font (size 1.27 1.27)) (justify right))
+    (property "Intersheet References" "${INTERSHEET_REFS}" (id 0) (at 204.8388 91.3606 0)
       (effects (font (size 1.27 1.27)) (justify right) hide)
     )
@@
     (effects (font (size 1.27 1.27)) (justify right))
     (property "Intersheet References" "${INTERSHEET_REFS}" (id 0) (at 167.5606 101.2312 90)
-      (effects (font (size 1.27 1.27)) (justify right) hide)
-    )
-  )
-  (global_label "5V" (shape input) (at 209.55 92.71 180) (fields_autoplaced)
-    (effects (font (size 1.27 1.27)) (justify right))
-    (property "Intersheet References" "${INTERSHEET_REFS}" (id 0) (at 204.8388 92.6306 0)
       (effects (font (size 1.27 1.27)) (justify right) hide)
     )
@@
     )
   )
-  (global_label "GNDUSB" (shape input) (at 157.48 144.78 270) (fields_autoplaced)
-    (effects (font (size 1.27 1.27)) (justify right))
-    (property "Intersheet References" "${INTERSHEET_REFS}" (id 0) (at 157.4006 154.8736 90)
-      (effects (font (size 1.27 1.27)) (justify right) hide)
-    )
-  )
-  (global_label "5VVA" (shape input) (at 170.18 116.84 0) (fields_autoplaced)
-    (effects (font (size 1.27 1.27)) (justify left))
-    (property "Intersheet References" "${INTERSHEET_REFS}" (id 0) (at 177.0683 116.7606 0)
-      (effects (font (size 1.27 1.27)) (justify left) hide)
+  (global_label "GNDUSB" (shape input) (at 156.21 120.65 180) (fields_autoplaced)
+    (effects (font (size 1.27 1.27)) (justify right))
+    (property "Intersheet References" "${INTERSHEET_REFS}" (id 0) (at 146.1164 120.5706 0)
+      (effects (font (size 1.27 1.27)) (justify right) hide)
+    )
+  )
+  (global_label "5VVA" (shape input) (at 156.21 118.11 180) (fields_autoplaced)
+    (effects (font (size 1.27 1.27)) (justify right))
+    (property "Intersheet References" "${INTERSHEET_REFS}" (id 0) (at 149.3217 118.1894 0)
+      (effects (font (size 1.27 1.27)) (justify right) hide)
     )
   )
@@
     )
   )
-  (symbol (lib_id "Connector:Screw_Terminal_01x02") (at 214.63 92.71 0) (unit 1)
-    (in_bom yes) (on_board yes) (fields_autoplaced)
-    (property "Reference" "Button5V1" (id 0) (at 217.17 92.7099 0)
-      (effects (font (size 1.27 1.27)) (justify left))
-    )
-    (property "Value" "Screw_Terminal_01x02" (id 1) (at 217.17 95.2499 0)
-      (effects (font (size 1.27 1.27)) (justify left))
-    )
-    (property "Footprint" "TerminalBlock:TerminalBlock_bornier-2_P5.08mm" (id 2) (at 214.63 92.71 0)
-      (effects (font (size 1.27 1.27)) hide)
-    )
-    (property "Datasheet" "~" (id 3) (at 214.63 92.71 0)
+  (global_label "GND" (shape input) (at 209.55 93.98 180) (fields_autoplaced)
+    (effects (font (size 1.27 1.27)) (justify right))
+    (property "Intersheet References" "${INTERSHEET_REFS}" (id 0) (at 203.2664 93.9006 0)
+      (effects (font (size 1.27 1.27)) (justify right) hide)
+    )
+  )
+  (symbol (lib_id "Connector:Screw_Terminal_01x02") (at 161.29 118.11 0) (unit 1)
+    (in_bom yes) (on_board yes) (fields_autoplaced)
+    (property "Reference" "USB1" (id 0) (at 163.83 118.1099 0)
+      (effects (font (size 1.27 1.27)) (justify left))
+    )
+    (property "Value" "Screw_Terminal_01x02" (id 1) (at 163.83 120.6499 0)
+      (effects (font (size 1.27 1.27)) (justify left))
+    )
+    (property "Footprint" "TerminalBlock:TerminalBlock_bornier-2_P5.08mm" (id 2) (at 161.29 118.11 0)
+      (effects (font (size 1.27 1.27)) hide)
+    )
+    (property "Datasheet" "~" (id 3) (at 161.29 118.11 0)
       (effects (font (size 1.27 1.27)) hide)
     )
@@
     (pin "2")
   )
+  (symbol (lib_id "Connector:Screw_Terminal_01x03") (at 214.63 93.98 0) (unit 1)
+    (in_bom yes) (on_board yes) (fields_autoplaced)
+    (property "Reference" "Button5V1" (id 0) (at 217.17 92.7099 0)
+      (effects (font (size 1.27 1.27)) (justify left))
+    )
+    (property "Value" "Screw_Terminal_01x03" (id 1) (at 217.17 95.2499 0)
+      (effects (font (size 1.27 1.27)) (justify left))
+    )
+    (property "Footprint" "TerminalBlock:TerminalBlock_bornier-3_P5.08mm" (id 2) (at 214.63 93.98 0)
+      (effects (font (size 1.27 1.27)) hide)
+    )
+    (property "Datasheet" "~" (id 3) (at 214.63 93.98 0)
+      (effects (font (size 1.27 1.27)) hide)
+    )
+    (pin "1")
+    (pin "2")
+    (pin "3")
+  )
   (symbol (lib_id "Device:C_Polarized") (at 194.31 82.55 270) (unit 1)
     (in_bom yes) (on_board yes) (fields_autoplaced)
@@
     (pin "1")
     (pin "2")
-  )
-  (symbol (lib_id "Connector:USB3_A") (at 157.48 127 0) (unit 1)
-    (in_bom yes) (on_board yes) (fields_autoplaced)
-    (property "Reference" "5VUSB1" (id 0) (at 157.48 107.95 0))
-    (property "Value" "USB3_A" (id 1) (at 157.48 110.49 0))
-    (property "Footprint" "Connector_USB:USB_A_CONNFLY_DS1095-WNR0" (id 2) (at 161.29 121.92 0)
-      (effects (font (size 1.27 1.27)) hide)
-    )
-    (property "Datasheet" "~" (id 3) (at 161.29 124.46 0)
-      (effects (font (size 1.27 1.27)) hide)
-    )
-    (pin "1")
-    (pin "4")
   )
   (symbol (lib_id "Device:C_Polarized") (at 194.31 55.88 270) (unit 1)
@@
       (reference "5VRegulator1") (unit 1) (value "LM7805_TO220") (footprint "Package_TO_SOT_THT:TO-220-3_Vertical")
     )
-    (path "/c2de80eb-de6e-402c-bde0-f2c12ca18548"
-      (reference "5VUSB1") (unit 1) (value "USB3_A") (footprint "Connector_USB:USB_A_CONNFLY_DS1095-WNR0")
-    )
     (path "/9335a357-224a-4bc6-b052-c3b76075508d"
       (reference "5VVoltamperimeter1") (unit 1) (value "Screw_Terminal_01x05") (footprint "TerminalBlock:TerminalBlock_bornier-5_P5.08mm")
     )
-    (path "/039f3315-a7e1-4670-9d91-eda7d93abebf"
-      (reference "Button5V1") (unit 1) (value "Screw_Terminal_01x02") (footprint "TerminalBlock:TerminalBlock_bornier-2_P5.08mm")
+    (path "/45875e59-c699-46c8-b157-7ea00437b45c"
+      (reference "Button5V1") (unit 1) (value "Screw_Terminal_01x03") (footprint "TerminalBlock:TerminalBlock_bornier-3_P5.08mm")
     )
     (path "/d9e9869d-e74b-4d48-9b17-fd243c0fc8b2"
@@
       (reference "Transformer1") (unit 1) (value "Screw_Terminal_01x02") (footprint "TerminalBlock:TerminalBlock_bornier-2_P5.08mm")
     )
-  )
+    (path "/01708a67-c98f-421c-90a8-5622374a8c4c"
+      (reference "USB1") (unit 1) (value "Screw_Terminal_01x02") (footprint "TerminalBlock:TerminalBlock_bornier-2_P5.08mm")
+    )
+  )
